File: lithium_ion_charging_block.sch (KiCad schematic (older format))
At the start: 19 parts, among them J1 10118194-0001LF, J2 Conn_01x02, Q1 Q_PMOS_DSG, U1 MCP73831-2-OT, U2 TPS61200DRC

Commit message: Added schematic and readme
Parts:
- R2: value R -> 330
Changed lines of the file:
@@
 P 4200 2150
 F 0 "R2" V 3993 2150 50  0000 C CNN
-F 1 "R" V 4084 2150 50  0000 C CNN
+F 1 "330" V 4200 2150 50  0000 C CNN
 F 2 "Resistor_SMD:R_0805_2012Metric_Pad1.15x1.40mm_HandSolder" V 4130 2150 50  0001 C CNN
 F 3 "~" H 4200 2150 50  0001 C CNN
